Commit message: Added gazebo tag and changed stl scale

File: urdf/robot.urdf (robot description, URDF)
Before this commit: robot robot_name, 7 links, 6 joints
Links:
- removed link front_left_wheel
- removed link laser
- removed link rear_left_wheel
- removed link rear_right_wheel
- link base: mass None -> 15.0; geometry collision box size=0.5 0.3 0.15; visual box size=0.5 0.3 0.15
- link base_link: mass None -> 0.1
- link front_right_wheel: mass None -> 1.0; geometry collision cylinder length=0.05 radius=0.1; visual mesh filename=package://robot_description/stl/blue_tyre_scaled.stl scale=1 1 1
Joints:
- removed joint front_left_wheel_joint
- removed joint laser_joint
- removed joint rear_left_wheel_joint
- removed joint rear_right_wheel_joint
- joint base_link_to_base: origin xyz=0.0 0.0 0.0 rpy=0.0 0.0 0.0 -> xyz=0 0 0 rpy=0 0 0
