Commit message: Added gazebo functionality

File: urdf/myrobot.urdf.xacro (robot description, xacro)
@@ -1,42 +1,21 @@
 <?xml version="1.0"?>
 <robot name="robot_name" xmlns:xacro="http://ros.org/wiki/xacro">
-    <!-- Materials remain the same -->
-    <material name="blue">
-        <color rgba="0 0 0.8 1" />
-    </material>
-    <material name="grey">
-        <color rgba="0.9 0.95 0.95 1.0" />
-    </material>
-    <material name="black">
-        <color rgba="0 0 0 1" />
-    </material>
-    <material name="green">
-        <color rgba="0.0 0.8 0.0 1.0" />
-    </material>
-    <!-- Properties -->
-    <xacro:property name="scale_stl" value="1 1 1" />
-    <xacro:property name="wheel_dist_x" value="0.21" />
-    <xacro:property name="wheel_dist_y" value="0.35" />
-    <xacro:property name="lidar_dist_x" value="0.363" />
-    <xacro:property name="lidar_dist_y" value="0" />
-    <xacro:property name="lidar_dist_z" value="0.239" />
-    <xacro:property name="pie" value="3.1415926" />
-    <!-- Wheel properties -->
-    <xacro:property name="wheel_radius" value="0.1" />
-    <xacro:property name="wheel_thickness" value="0.05" />
-    <xacro:property name="wheel_mass" value="1.0" />
-    <!-- Base properties -->
-    <xacro:property name="base_mass" value="15.0" />
-    <xacro:property name="base_length" value="0.5" />
-    <xacro:property name="base_width" value="0.3" />
-    <xacro:property name="base_height" value="0.15" />
+    <xacro:include filename="properties.xacro" />
     <!-- Root Link -->
+    <link name="base_footprint">
+    </link>
     <link name="base_link">
     </link>
+    <joint name="base_foot_to_base_link" type="fixed">
+        <parent link="base_link"/>
+        <child link="base_footprint"/>
+        <origin xyz="0.0 0.0 0.0" rpy="0.0 0.0 0.0"/>
+    </joint>
     <link name="base">
         <visual>
-            <origin xyz="0.0 0.0 0.0" rpy="0.0 0.0 0.0" />
+            <origin xyz="0.0 0.0 0" rpy="0.0 0.0 0.0" />
             <geometry>
-                <mesh filename="package://myrobot_description/stl/base.stl" scale="${scale_stl}" />
+                <mesh filename="file://$(find myrobot_description)/meshes/base.stl"
+                    scale="${scale_stl}" />
             </geometry>
             <material name="grey" />
@@ -63,7 +42,9 @@
         <link name="${prefix}_wheel">
             <visual>
-                <origin rpy="0 0 0" xyz="0 0 0" />
+                <origin xyz="0 0 0" rpy="0 0 0" />
                 <geometry>
-                    <mesh filename="package://myrobot_description/stl/blue_tyre.stl"
+                    <!-- <mesh filename="package://myrobot_description/meshes/blue_tyre.stl"
+                        scale="${scale_stl}" /> -->
+                    <mesh filename="file://$(find myrobot_description)/meshes/blue_tyre.stl"
                         scale="${scale_stl}" />
                 </geometry>
@@ -71,7 +52,9 @@
             </visual>
             <collision>
-                <origin rpy="${pi/2} 0 0" xyz="0 0 0" />
+                <origin rpy="0 0 0" xyz="0 0 0" />
                 <geometry>
-                    <cylinder radius="${wheel_radius}" length="${wheel_thickness}" />
+                    <!-- <cylinder radius="${wheel_radius}" length="${wheel_thickness}" /> -->
+                    <mesh filename="file://$(find myrobot_description)/meshes/blue_tyre.stl"
+                        scale="${scale_stl}" />
                 </geometry>
             </collision>
@@ -83,15 +66,13 @@
                     ixy="0"
                     ixz="0"
-                    iyy="${wheel_mass * (3 * wheel_radius * wheel_radius + wheel_thickness * wheel_thickness) / 12}"
+                    iyy="${wheel_mass * wheel_radius * wheel_radius / 2}"
                     iyz="0"
-                    izz="${wheel_mass * wheel_radius * wheel_radius / 2}" />
+                    izz="${wheel_mass * (3 * wheel_radius * wheel_radius + wheel_thickness * wheel_thickness) / 12}" />
             </inertial>
         </link>
         <gazebo reference="${prefix}_wheel">
             <material>Gazebo/Black</material>
-            <mu1 value="1.0" />
-            <mu2 value="1.0" />
-            <kp value="10000000.0" />
-            <kd value="1.0" />
+            <mu1 value="0.7" />
+            <mu2 value="0.7" />
         </gazebo>
     </xacro:macro>
@@ -105,5 +86,5 @@
         <parent link="base_link" />
         <child link="base" />
-        <origin xyz="0.0 0.0 0.0" rpy="0.0 0.0 0.0" />
+        <origin xyz="0.0 0.0 ${wheel_radius}" rpy="0.0 0.0 0.0" />
     </joint>
     <joint name="front_right_wheel_joint" type="continuous">
@@ -136,5 +117,6 @@
             <origin rpy="0 0 0" xyz="0 0 0" />
             <geometry>
-                <mesh filename="package://myrobot_description/stl/mid_360.stl" scale="${scale_stl}" />
+                <mesh filename="file://$(find myrobot_description)/meshes/mid_360.stl"
+                    scale="${scale_stl}" />
             </geometry>
             <material name="blue" />
@@ -159,6 +141,7 @@
         <child link="laser" />
     </joint>
-    <gazebo reference="laser">
-        <material>Gazebo/Blue</material>
-    </gazebo>
+    <xacro:include filename="laser.urdf.xacro" />
+    <xacro:include filename="gazebo_control.xacro" />
+    <xacro:include filename="imu.urdf.xacro" />
+    <xacro:imu />
 </robot>
